Commit message: Change HeadPitch to 20.0 degrees

File: pepper_description/urdf/pepper1.0_generated_urdf/pepper_head.xacro (robot description, xacro)
@@ -22,5 +22,5 @@
 		<parent link="Neck"/>
 		<child link="Head"/>
-		<origin rpy="0 0 0" xyz="0 0 0"/>
+		<origin rpy="0 0.3490 0" xyz="0 0 0"/>
 		<axis xyz="0 1.0 0"/>
 		<limit effort="2.666" lower="-0.706858" upper="0.637045" velocity="9.22756"/>

Commit message: Change height of table, HeadPitch and HeadYaw

File: pepper_description/urdf/pepper1.0_generated_urdf/pepper_head.xacro (robot description, xacro)
@@ -7,5 +7,5 @@
 		<parent link="torso"/>
 		<child link="Neck"/>
-		<origin rpy="0 0 0" xyz="-0.038 0 0.1699"/>
+		<origin rpy="0 0 -0.1" xyz="-0.038 0 0.1699"/>
 		<axis xyz="0 0 1.0"/>
 		<limit effort="5.428" lower="-2.08567" upper="2.08567" velocity="7.33998"/>
@@ -22,5 +22,5 @@
 		<parent link="Neck"/>
 		<child link="Head"/>
-		<origin rpy="0 0.3490 0" xyz="0 0 0"/>
+		<origin rpy="0 0.05 0" xyz="0 0 0"/>
 		<axis xyz="0 1.0 0"/>
 		<limit effort="2.666" lower="-0.706858" upper="0.637045" velocity="9.22756"/>

Commit message: Change HeadYaw and HeadPitch

File: pepper_description/urdf/pepper1.0_generated_urdf/pepper_head.xacro (robot description, xacro)
@@ -7,5 +7,6 @@
 		<parent link="torso"/>
 		<child link="Neck"/>
-		<origin rpy="0 0 -0.1" xyz="-0.038 0 0.1699"/>
+		<origin rpy="0 0 -0.34906585039" xyz="-0.038 0 0.1699"/>
+		<!-- 20 degrees -->
 		<axis xyz="0 0 1.0"/>
 		<limit effort="5.428" lower="-2.08567" upper="2.08567" velocity="7.33998"/>
@@ -22,5 +23,6 @@
 		<parent link="Neck"/>
 		<child link="Head"/>
-		<origin rpy="0 0.05 0" xyz="0 0 0"/>
+		<origin rpy="0 0.17453292519 0" xyz="0 0 0"/>
+		<!-- 10 degrees -->
 		<axis xyz="0 1.0 0"/>
 		<limit effort="2.666" lower="-0.706858" upper="0.637045" velocity="9.22756"/>
