Commit message: Add table model

File: pepper_description/urdf/pepper1.0_generated_urdf/pepper_arms.xacro (robot description, xacro)
@@ -7,5 +7,5 @@
 		<parent link="torso"/>
 		<child link="LShoulder"/>
-		<origin rpy="0 0 0" xyz="-0.057 0.14974 0.08682"/>
+		<origin rpy="0 0.52359877559 0" xyz="-0.057 0.14974 0.08682"/>
 		<axis xyz="0 1.0 0"/>
 		<limit effort="5.428" lower="-2.08567" upper="2.08567" velocity="7.33998"/>
@@ -95,5 +95,5 @@
 		<parent link="torso"/>
 		<child link="RShoulder"/>
-		<origin rpy="0 0 0" xyz="-0.057 -0.14974 0.08682"/>
+		<origin rpy="0 0.52359877559 0" xyz="-0.057 -0.14974 0.08682"/>
 		<axis xyz="0 1.0 0"/>
 		<limit effort="5.428" lower="-2.08567" upper="2.08567" velocity="7.33998"/>

Commit message: Change x and y position of RightArm and cube and Head

File: pepper_description/urdf/pepper1.0_generated_urdf/pepper_arms.xacro (robot description, xacro)
@@ -95,5 +95,6 @@
 		<parent link="torso"/>
 		<child link="RShoulder"/>
-		<origin rpy="0 0.52359877559 0" xyz="-0.057 -0.14974 0.08682"/>
+		<origin rpy="0 0.61086523819 0" xyz="-0.057 -0.14974 0.08682"/>
+		<!-- 35 degrees -->
 		<axis xyz="0 1.0 0"/>
 		<limit effort="5.428" lower="-2.08567" upper="2.08567" velocity="7.33998"/>
@@ -110,5 +111,6 @@
 		<parent link="RShoulder"/>
 		<child link="RBicep"/>
-		<origin rpy="0 0 0" xyz="0 0 0"/>
+		<origin rpy="0 0 -0.34906585039" xyz="0 0 0"/>
+		<!-- -20 degrees -->
 		<axis xyz="0 0 1.0"/>
 		<limit effort="2.666" lower="-1.56207" upper="-0.00872665" velocity="9.22756"/>
