Commit message: [change] Initial position of models to reachable for Pepper. Pepperの手が届く範囲にオブジェクトの初期位置を変更

File: my_pepper_description/urdf/pepper1.0_generated_urdf/pepper_arms.xacro (robot description, xacro)
@@ -95,6 +95,6 @@
 		<parent link="torso"/>
 		<child link="RShoulder"/>
-		<origin rpy="0 0.61086523819 0" xyz="-0.057 -0.14974 0.08682"/>
-		<!-- 35 degrees -->
+		<origin rpy="0 0.6981317008 0" xyz="-0.057 -0.14974 0.08682"/>
+		<!-- 40 degrees -->
 		<axis xyz="0 1.0 0"/>
 		<limit effort="5.428" lower="-2.08567" upper="2.08567" velocity="7.33998"/>
@@ -111,6 +111,6 @@
 		<parent link="RShoulder"/>
 		<child link="RBicep"/>
-		<origin rpy="0 0 -0.34906585039" xyz="0 0 0"/>
-		<!-- -20 degrees -->
+		<origin rpy="0 0 -0.6981317008" xyz="0 0 0"/>
+		<!-- -40 degrees -->
 		<axis xyz="0 0 1.0"/>
 		<limit effort="2.666" lower="-1.56207" upper="-0.00872665" velocity="9.22756"/>
