Commit message: [change] limits of RShoulderRoll

File: src/my_pepper_description/urdf/pepper1.0_generated_urdf/pepper_arms.xacro (robot description, xacro)
@@ -114,5 +114,5 @@
 		<!-- -40 degrees -->
 		<axis xyz="0 0 1.0"/>
-		<limit effort="2.666" lower="-1.56207" upper="-0.00872665" velocity="9.22756"/>
+		<limit effort="2.666" lower="-1.56207" upper="1.00872665" velocity="9.22756"/>
 	</joint>
 	<link name="RBicep">
@@ -127,5 +127,5 @@
 		<parent link="RBicep"/>
 		<child link="RElbow"/>
-		<origin rpy="0 -0.157079 0" xyz="0.1812 -0.015 0.00013"/>
+		<origin rpy="0 0 0" xyz="0.1812 -0.015 0.00013"/>
 		<axis xyz="1.0 0 0"/>
 		<limit effort="5.428" lower="-2.08567" upper="2.08567" velocity="7.33998"/>

File: src/my_pepper_description/urdf/pepper1.0_generated_urdf/pepper_robot.xacro (robot description, xacro)
@@ -10,5 +10,5 @@
 	<xacro:include filename="pepper_arms.xacro"/>
 	<xacro:include filename="pepper_sensors.xacro"/>
-	<xacro:include filename="pepper_fingers.xacro"/>
+	<!-- <xacro:include filename="pepper_fingers.xacro"/> -->
 	<xacro:include filename="pepper_wheels.xacro"/>
 	<xacro:include filename="pepperGazebo.xacro"/>

Commit message: [add] with human

File: src/my_pepper_description/urdf/pepper1.0_generated_urdf/pepper_arms.xacro (robot description, xacro)
@@ -157,5 +157,5 @@
 		<parent link="RForeArm"/>
 		<child link="r_wrist"/>
-		<origin rpy="0 0 0" xyz="0.15 0 0"/>
+		<origin rpy="0.95 0 0" xyz="0.15 0 0"/>
 		<axis xyz="1.0 0 0"/>
 		<limit effort="0.2014" lower="-1.82387" upper="1.82387" velocity="17.3835"/>
